Commit message: notes added

File: src/rsp/week04_description/urdf/mylink.xacro (robot description, xacro)
@@ -5,5 +5,5 @@
             <inertial>
                 <mass value="1"/>
-                <origin xyz="0.0 0.0 0.0" rpy="0.0 0.0 0.0"/>
+                <origin xyz="0 0 0" rpy="0 0 0"/>
                 <inertia ixx="1" ixy="0.0" ixz="0.0" iyy="1" iyz="0.0" izz="1"/>
             </inertial>
@@ -11,11 +11,11 @@
                 <origin xyz="0 0 0.5" rpy="0 0 0"/>
                 <geometry>
-                    <box size="0.1 0.1 1"/>
+                    <box size="0.4 0.4 1"/>
                 </geometry>
             </visual>
             <collision>
-                <origin xyz="0.0 0.0 -0.5" rpy="0.0 0.0 0.0"/>
+                <origin xyz="0 0 0.5" rpy="0 0 0"/>
                 <geometry>
-                    <box size="0.4 0.4 1"/>
+                    <box size="0.5 0.5 1.5"/>
                 </geometry>
             </collision>
@@ -23,5 +23,5 @@
     </xacro:macro>
     <!-- instead of writing same code for different links, we can reuse the code like above -->
-    <xacro:macro name="toollink">
+    <!-- <xacro:macro name="toollink">
         <link name="tool">
             <visual>
@@ -32,4 +32,4 @@
             </visual>
         </link>
-    </xacro:macro>
+    </xacro:macro> -->
 </robot>

File: src/rsp/week04_description/urdf/simple_robot-v1.urdf.xacro (robot description, xacro)
@@ -2,5 +2,5 @@
     <xacro:include filename="$(find week04_description)/urdf/mylink.xacro"/>
     <xacro:worldlink/>
-    <xacro:toollink/>
+    <!-- <xacro:toollink/>
     <joint name="q1" type="revolute">
         <origin xyz="0 0 0.5" rpy=" 0 0 0"/>
@@ -9,4 +9,4 @@
         <axis xyz="0 0 1"/>
         <limit lower="-1" upper="1" effort="1" velocity="1"/>
-    </joint>
+    </joint> -->
 </robot>
