Commit message: backup

File: src/assignment5/edumip_description/urdf/edumip.xacro (robot description, xacro)
@@ -70,5 +70,5 @@
             <parent link="base_link"/>
             <child link="left_wheel"/>
-            <axis xyz="0 0 1"/>
+            <axis xyz="0 1 0"/>
         </joint>
         <joint name="right_joint" type="continuous">
@@ -76,5 +76,5 @@
             <parent link="base_link"/>
             <child link="right_wheel"/>
-            <axis xyz="0 0 1"/>
+            <axis xyz="0 1 0"/>
         </joint>
     </xacro:macro>
